File: iot-badge-vhf/iot-badge-vhf.kicad_sch (KiCad schematic)
At the start: 62 parts, among them J1 USB_C_Receptacle_USB2.0, J2 Wire ANT, Q1 BC847, Q2 BC847, Q3 BC847, SW1 SW_Push, SW2 SW_Push, SW3 SW_Push, SW4 SW_Push, SW5 SW_Push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

Commit message: created iot badge VHF
Other:
- title: IoT Badge -> IoT Badge VHF
Changed lines of the file:
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@@
   (paper "A4")
   (title_block
-    (title "IoT Badge")
+    (title "IoT Badge VHF")
     (company "Galopago")
   )
