File: iot-badge-915/iot-badge-915.kicad_pcb (KiCad board)
At the start: 2 copper layers, 70 x 100 mm, 64 parts, among them J1 USB_C_Receptacle_USB2.0, J2 Wire ANT, Q1 BC847, Q2 BC847, Q3 BC847, SW1 SW_Push, SW2 SW_Push, SW3 SW_Push, SW4 SW_Push, SW5 SW_Push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

Commit message: 915 version finished
Parts:
- removed L1: L, Inductor_SMD:L_0805_2012Metric_Pad1.05x1.20mm_HandSolder
- added C12: C, Capacitor_SMD:C_0805_2012Metric_Pad1.18x1.45mm_HandSolder, F.Cu at (105.0, 71.8)
- AE1: value Antenna 433 -> Antenna 915; footprint RF_PCB_Antenna:Micrel_Heli_2 -> RF_PCB_Antenna:Micrel_916_ant_6
- moved AE1 7.02 mm to (116.2, 61.0)
Routing:
- net Net-(AE1-Pad1): track 3.26 -> 8.56 mm
- net Earth: vias 96 -> 104
Other:
- board text added: "IoT Badge V 00 915"
- board text removed: "IoT Badge V 00"
