File: iot-badge-915/iot-badge-915.kicad_sch (KiCad schematic)
At the start: 62 parts, among them J1 USB_C_Receptacle_USB2.0, J2 Wire ANT, Q1 BC847, Q2 BC847, Q3 BC847, SW1 SW_Push, SW2 SW_Push, SW3 SW_Push, SW4 SW_Push, SW5 SW_Push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

Commit message: created iot 433 and 915 versions (renamed)
Other:
- title: IoT Badge VHF -> IoT Badge 915
Changed lines of the file:
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@@
   (paper "A4")
   (title_block
-    (title "IoT Badge VHF")
+    (title "IoT Badge 915")
     (company "Galopago")
   )

Commit message: 915 version finished
Parts:
- removed AE1: Antenna 433, RF_PCB_Antenna:Micrel_Heli_2, symbol Device:Antenna
- removed L1: L, Inductor_SMD:L_0805_2012Metric_Pad1.05x1.20mm_HandSolder, symbol Device:L
- added AE1: Antenna 915, RF_PCB_Antenna:Micrel_916_ant_6, symbol Device:Antenna_Dipole
- added C12: C, Capacitor_SMD:C_0805_2012Metric_Pad1.18x1.45mm_HandSolder, symbol Device:C
Connections:
- net Earth: now also AE1.2, C12.1
- net at C9.1: now also AE1.1, C12.2
Changed lines of the file:
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@@
+    (stroke (width 0) (type default) (color 0 0 0 0))
+  )
+  (wire (pts (xy 184.15 76.2) (xy 184.15 77.47))
     (stroke (width 0) (type default) (color 0 0 0 0))
   )
@@
     (pin "1")
   )
-  (symbol (lib_id "Device:Antenna") (at 181.61 71.12 0) (unit 1)
-    (in_bom yes) (on_board yes) (fields_autoplaced)
-    (property "Reference" "AE1" (id 0) (at 184.15 70.4849 0)
-      (effects (font (size 1.27 1.27)) (justify left))
-    )
-    (property "Value" "Antenna 433" (id 1) (at 184.15 73.0249 0)
-      (effects (font (size 1.27 1.27)) (justify left))
-    )
-    (property "Footprint" "RF_PCB_Antenna:Micrel_Heli_2" (id 2) (at 181.61 71.12 0)
-      (effects (font (size 1.27 1.27)) hide)
-    )
-    (property "Datasheet" "~" (id 3) (at 181.61 71.12 0)
-      (effects (font (size 1.27 1.27)) hide)
-    )
-    (pin "1")
-  )
   (symbol (lib_id "power:+BATT") (at 207.01 25.4 0) (unit 1)
     (in_bom yes) (on_board yes) (fields_autoplaced)
@@
     (pin "2")
     (pin "3")
+  )
+  (symbol (lib_id "Device:Antenna_Dipole") (at 181.61 71.12 0) (unit 1)
+    (in_bom yes) (on_board yes) (fields_autoplaced)
+    (property "Reference" "AE1" (id 0) (at 187.96 72.3899 0)
+      (effects (font (size 1.27 1.27)) (justify left))
+    )
+    (property "Value" "Antenna 915" (id 1) (at 187.96 74.9299 0)
+      (effects (font (size 1.27 1.27)) (justify left))
+    )
+    (property "Footprint" "RF_PCB_Antenna:Micrel_916_ant_6" (id 2) (at 181.61 71.12 0)
+      (effects (font (size 1.27 1.27)) hide)
+    )
+    (property "Datasheet" "~" (id 3) (at 181.61 71.12 0)
+      (effects (font (size 1.27 1.27)) hide)
+    )
+    (pin "1")
+    (pin "2")
   )
   (symbol (lib_id "Device:R") (at 114.3 49.53 0) (unit 1)
@@
     (pin "1")
   )
-  (symbol (lib_id "Device:L") (at 181.61 85.09 0) (unit 1)
-    (in_bom yes) (on_board yes) (fields_autoplaced)
-    (property "Reference" "L1" (id 0) (at 182.88 83.8199 0)
-      (effects (font (size 1.27 1.27)) (justify left))
-    )
-    (property "Value" "L" (id 1) (at 182.88 86.3599 0)
-      (effects (font (size 1.27 1.27)) (justify left))
-    )
-    (property "Footprint" "Inductor_SMD:L_0805_2012Metric_Pad1.05x1.20mm_HandSolder" (id 2) (at 181.61 85.09 0)
+  (symbol (lib_id "Device:C") (at 181.61 85.09 180) (unit 1)
+    (in_bom yes) (on_board yes) (fields_autoplaced)
+    (property "Reference" "C12" (id 0) (at 185.42 83.8199 0)
+      (effects (font (size 1.27 1.27)) (justify right))
+    )
+    (property "Value" "C" (id 1) (at 185.42 86.3599 0)
+      (effects (font (size 1.27 1.27)) (justify right))
+    )
+    (property "Footprint" "Capacitor_SMD:C_0805_2012Metric_Pad1.18x1.45mm_HandSolder" (id 2) (at 180.6448 81.28 0)
       (effects (font (size 1.27 1.27)) hide)
     )
@@
     )
     (property "Datasheet" "~" (id 3) (at 110.49 161.29 0)
+      (effects (font (size 1.27 1.27)) hide)
+    )
+    (pin "1")
+  )
+  (symbol (lib_id "power:Earth") (at 184.15 77.47 0) (unit 1)
+    (in_bom yes) (on_board yes) (fields_autoplaced)
+    (property "Reference" "#PWR0121" (id 0) (at 184.15 83.82 0)
+      (effects (font (size 1.27 1.27)) hide)
+    )
+    (property "Value" "Earth" (id 1) (at 184.15 81.28 0)
+      (effects (font (size 1.27 1.27)) hide)
+    )
+    (property "Footprint" "" (id 2) (at 184.15 77.47 0)
+      (effects (font (size 1.27 1.27)) hide)
+    )
+    (property "Datasheet" "~" (id 3) (at 184.15 77.47 0)
       (effects (font (size 1.27 1.27)) hide)
     )
@@
       (reference "#PWR0120") (unit 1) (value "+3V3") (footprint "")
     )
+    (path "/a6cc9813-9dd2-4d83-8985-94227857afe5"
+      (reference "#PWR0121") (unit 1) (value "Earth") (footprint "")
+    )
     (path "/b5cbfbc3-2fc4-46f9-b933-de18f4b24ce3"
       (reference "#PWR0122") (unit 1) (value "Earth") (footprint "")
@@
       (reference "#PWR0137") (unit 1) (value "+3V3") (footprint "")
     )
-    (path "/17a036a7-3c7d-4750-8cd7-b5f99a19695c"
-      (reference "AE1") (unit 1) (value "Antenna 433") (footprint "RF_PCB_Antenna:Micrel_Heli_2")
+    (path "/3eadd3f7-174c-4ff3-9be3-e1f91e060ec2"
+      (reference "AE1") (unit 1) (value "Antenna 915") (footprint "RF_PCB_Antenna:Micrel_916_ant_6")
     )
     (path "/2c63cd38-91d8-4cab-a48b-fb9392e1f840"
@@
       (reference "C11") (unit 1) (value "100uF") (footprint "Capacitor_Tantalum_SMD:CP_EIA-2012-15_AVX-P_Pad1.30x1.05mm_HandSolder")
     )
+    (path "/878dc4bf-ba06-4686-adac-a3b35cd3741d"
+      (reference "C12") (unit 1) (value "C") (footprint "Capacitor_SMD:C_0805_2012Metric_Pad1.18x1.45mm_HandSolder")
+    )
     (path "/2dbc282c-a4c9-44f2-b1b6-9acbf2576b02"
       (reference "D1") (unit 1) (value "LED_RGB") (footprint "LED_SMD:LED_RGB_5050-6")
@@
       (reference "JP1") (unit 1) (value "Jumper_3_Bridged12") (footprint "Jumper:SolderJumper-3_P1.3mm_Bridged12_RoundedPad1.0x1.5mm_NumberLabels")
     )
-    (path "/8697a252-c3b7-4af5-869c-16261fab2989"
-      (reference "L1") (unit 1) (value "L") (footprint "Inductor_SMD:L_0805_2012Metric_Pad1.05x1.20mm_HandSolder")
-    )
     (path "/5206bb1c-8aa7-4043-9932-e730bc472f2a"

Commit message: changed ir leds polarity, PSU silk and bypass jumper
Parts:
- added JP2: SolderJumper_2_Open, Jumper:SolderJumper-2_P1.3mm_Open_RoundedPad1.0x1.5mm, symbol Jumper:SolderJumper_2_Open
Connections:
- net +3V3: no longer D6.2 (A)
- net +BATT: now also JP2.1 (A)
- net Earth: now also D6.1 (K)
- net at R11.2, SW9.1 (A), U6.2 (VOUT): now also JP2.2 (B)
- net at D5.1 (K): now also D6.2 (A); no longer R18.1
- net at D5.2 (A): now also R18.1; no longer D6.1 (K)
Other:
- moved on the sheet: D5, D6, R18
Changed lines of the file:
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@@
   (junction (at 114.3 55.88) (diameter 0) (color 0 0 0 0)
+  )
+  (junction (at 218.44 26.67) (diameter 0) (color 0 0 0 0)
   )
   (junction (at 104.14 176.53) (diameter 0) (color 0 0 0 0)
@@
     (stroke (width 0) (type default) (color 0 0 0 0))
   )
-  (wire (pts (xy 254 64.77) (xy 254 66.04))
-    (stroke (width 0) (type default) (color 0 0 0 0))
-  )
   (wire (pts (xy 138.43 158.75) (xy 146.05 158.75))
     (stroke (width 0) (type default) (color 0 0 0 0))
@@
     (stroke (width 0) (type default) (color 0 0 0 0))
   )
+  (wire (pts (xy 256.54 54.61) (xy 256.54 55.88))
+    (stroke (width 0) (type default) (color 0 0 0 0))
+  )
   (wire (pts (xy 148.59 121.92) (xy 148.59 99.06))
     (stroke (width 0) (type default) (color 0 0 0 0))
@@
     (stroke (width 0) (type default) (color 0 0 0 0))
   )
-  (wire (pts (xy 254 55.88) (xy 254 57.15))
-    (stroke (width 0) (type default) (color 0 0 0 0))
-  )
   (wire (pts (xy 128.27 149.86) (xy 128.27 151.13))
     (stroke (width 0) (type default) (color 0 0 0 0))
@@
     (stroke (width 0) (type default) (color 0 0 0 0))
   )
-  (wire (pts (xy 254 73.66) (xy 254 74.93))
-    (stroke (width 0) (type default) (color 0 0 0 0))
-  )
   (wire (pts (xy 138.43 156.21) (xy 142.24 156.21))
     (stroke (width 0) (type default) (color 0 0 0 0))
@@
     (stroke (width 0) (type default) (color 0 0 0 0))
   )
-  (wire (pts (xy 219.71 26.67) (xy 215.9 26.67))
+  (wire (pts (xy 219.71 26.67) (xy 218.44 26.67))
     (stroke (width 0) (type default) (color 0 0 0 0))
   )
@@
     (stroke (width 0) (type default) (color 0 0 0 0))
   )
+  (wire (pts (xy 241.3 17.78) (xy 241.3 25.4))
+    (stroke (width 0) (type default) (color 0 0 0 0))
+  )
   (wire (pts (xy 254 29.21) (xy 251.46 29.21))
     (stroke (width 0) (type default) (color 0 0 0 0))
@@
     (stroke (width 0) (type default) (color 0 0 0 0))
   )
-  (wire (pts (xy 251.46 74.93) (xy 254 74.93))
+  (wire (pts (xy 255.27 54.61) (xy 256.54 54.61))
     (stroke (width 0) (type default) (color 0 0 0 0))
   )
@@
     (stroke (width 0) (type default) (color 0 0 0 0))
   )
+  (wire (pts (xy 256.54 72.39) (xy 256.54 73.66))
+    (stroke (width 0) (type default) (color 0 0 0 0))
+  )
   (wire (pts (xy 43.18 162.56) (xy 58.42 162.56))
     (stroke (width 0) (type default) (color 0 0 0 0))
@@
     (stroke (width 0) (type default) (color 0 0 0 0))
   )
+  (wire (pts (xy 218.44 17.78) (xy 218.44 26.67))
+    (stroke (width 0) (type default) (color 0 0 0 0))
+  )
   (wire (pts (xy 171.45 80.01) (xy 167.64 80.01))
     (stroke (width 0) (type default) (color 0 0 0 0))
@@
     (stroke (width 0) (type default) (color 0 0 0 0))
   )
+  (wire (pts (xy 223.52 17.78) (xy 218.44 17.78))
+    (stroke (width 0) (type default) (color 0 0 0 0))
+  )
   (wire (pts (xy 167.64 80.01) (xy 167.64 83.82))
     (stroke (width 0) (type default) (color 0 0 0 0))
@@
     (stroke (width 0) (type default) (color 0 0 0 0))
   )
+  (wire (pts (xy 231.14 17.78) (xy 241.3 17.78))
+    (stroke (width 0) (type default) (color 0 0 0 0))
+  )
   (wire (pts (xy 115.57 176.53) (xy 115.57 177.8))
     (stroke (width 0) (type default) (color 0 0 0 0))
@@
     (stroke (width 0) (type default) (color 0 0 0 0))
   )
+  (wire (pts (xy 256.54 63.5) (xy 256.54 64.77))
+    (stroke (width 0) (type default) (color 0 0 0 0))
+  )
   (wire (pts (xy 64.77 76.2) (xy 80.01 76.2))
     (stroke (width 0) (type default) (color 0 0 0 0))
@@
     (stroke (width 0) (type default) (color 0 0 0 0))
   )
-  (wire (pts (xy 241.3 74.93) (xy 243.84 74.93))
+  (wire (pts (xy 245.11 54.61) (xy 247.65 54.61))
     (stroke (width 0) (type default) (color 0 0 0 0))
   )
@@
   )
   (wire (pts (xy 54.61 173.99) (xy 54.61 154.94))
+    (stroke (width 0) (type default) (color 0 0 0 0))
+  )
+  (wire (pts (xy 218.44 26.67) (xy 215.9 26.67))
     (stroke (width 0) (type default) (color 0 0 0 0))
   )
@@
     (effects (font (size 1.27 1.27)) (justify left bottom))
   )
-  (label "IRLED-2" (at 241.3 74.93 180)
+  (label "IRLED-2" (at 245.11 54.61 180)
     (effects (font (size 1.27 1.27)) (justify right bottom))
   )
@@
     )
     (property "Datasheet" "~" (id 3) (at 263.906 113.03 0)
+      (effects (font (size 1.27 1.27)) hide)
+    )
+    (pin "1")
+    (pin "2")
+  )
+  (symbol (lib_id "Jumper:SolderJumper_2_Open") (at 227.33 17.78 0) (unit 1)
+    (in_bom yes) (on_board yes)
+    (property "Reference" "JP2" (id 0) (at 227.33 13.97 0))
+    (property "Value" "SolderJumper_2_Open" (id 1) (at 227.33 15.24 0))
+    (property "Footprint" "Jumper:SolderJumper-2_P1.3mm_Open_RoundedPad1.0x1.5mm" (id 2) (at 227.33 17.78 0)
+      (effects (font (size 1.27 1.27)) hide)
+    )
+    (property "Datasheet" "~" (id 3) (at 227.33 17.78 0)
       (effects (font (size 1.27 1.27)) hide)
     )
@@
     (pin "2")
   )
-  (symbol (lib_id "Device:LED") (at 254 69.85 90) (unit 1)
-    (in_bom yes) (on_board yes)
-    (property "Reference" "D5" (id 0) (at 261.62 69.85 0))
-    (property "Value" "IRLED" (id 1) (at 259.08 69.85 0))
-    (property "Footprint" "LED_SMD:LED_0805_2012Metric_Pad1.15x1.40mm_HandSolder" (id 2) (at 254 69.85 0)
-      (effects (font (size 1.27 1.27)) hide)
-    )
-    (property "Datasheet" "~" (id 3) (at 254 69.85 0)
+  (symbol (lib_id "power:Earth") (at 256.54 73.66 0) (unit 1)
+    (in_bom yes) (on_board yes) (fields_autoplaced)
+    (property "Reference" "#PWR0137" (id 0) (at 256.54 80.01 0)
+      (effects (font (size 1.27 1.27)) hide)
+    )
+    (property "Value" "Earth" (id 1) (at 256.54 77.47 0)
+      (effects (font (size 1.27 1.27)) hide)
+    )
+    (property "Footprint" "" (id 2) (at 256.54 73.66 0)
+      (effects (font (size 1.27 1.27)) hide)
+    )
+    (property "Datasheet" "~" (id 3) (at 256.54 73.66 0)
+      (effects (font (size 1.27 1.27)) hide)
+    )
+    (pin "1")
+  )
+  (symbol (lib_id "Device:LED") (at 256.54 59.69 90) (unit 1)
+    (in_bom yes) (on_board yes)
+    (property "Reference" "D5" (id 0) (at 264.16 59.69 0))
+    (property "Value" "IRLED" (id 1) (at 261.62 59.69 0))
+    (property "Footprint" "LED_SMD:LED_0805_2012Metric_Pad1.15x1.40mm_HandSolder" (id 2) (at 256.54 59.69 0)
+      (effects (font (size 1.27 1.27)) hide)
+    )
+    (property "Datasheet" "~" (id 3) (at 256.54 59.69 0)
       (effects (font (size 1.27 1.27)) hide)
     )
@@
     (pin "2")
   )
-  (symbol (lib_id "power:+3V3") (at 254 55.88 0) (unit 1)
-    (in_bom yes) (on_board yes)
-    (property "Reference" "#PWR0137" (id 0) (at 254 59.69 0)
-      (effects (font (size 1.27 1.27)) hide)
-    )
-    (property "Value" "+3V3" (id 1) (at 254 50.8 0))
-    (property "Footprint" "" (id 2) (at 254 55.88 0)
-      (effects (font (size 1.27 1.27)) hide)
-    )
-    (property "Datasheet" "" (id 3) (at 254 55.88 0)
-      (effects (font (size 1.27 1.27)) hide)
-    )
-    (pin "1")
-  )
-  (symbol (lib_id "Device:LED") (at 254 60.96 90) (unit 1)
-    (in_bom yes) (on_board yes)
-    (property "Reference" "D6" (id 0) (at 261.62 60.96 0))
-    (property "Value" "IRLED" (id 1) (at 259.08 60.96 0))
-    (property "Footprint" "LED_SMD:LED_0805_2012Metric_Pad1.15x1.40mm_HandSolder" (id 2) (at 254 60.96 0)
-      (effects (font (size 1.27 1.27)) hide)
-    )
-    (property "Datasheet" "~" (id 3) (at 254 60.96 0)
+  (symbol (lib_id "Device:LED") (at 256.54 68.58 90) (unit 1)
+    (in_bom yes) (on_board yes)
+    (property "Reference" "D6" (id 0) (at 264.16 68.58 0))
+    (property "Value" "IRLED" (id 1) (at 261.62 68.58 0))
+    (property "Footprint" "LED_SMD:LED_0805_2012Metric_Pad1.15x1.40mm_HandSolder" (id 2) (at 256.54 68.58 0)
+      (effects (font (size 1.27 1.27)) hide)
+    )
+    (property "Datasheet" "~" (id 3) (at 256.54 68.58 0)
       (effects (font (size 1.27 1.27)) hide)
     )
@@
     (pin "3")
   )
-  (symbol (lib_id "Device:R") (at 247.65 74.93 270) (unit 1)
-    (in_bom yes) (on_board yes) (fields_autoplaced)
-    (property "Reference" "R18" (id 0) (at 247.65 68.58 90))
-    (property "Value" "500" (id 1) (at 247.65 71.12 90))
-    (property "Footprint" "Resistor_SMD:R_0805_2012Metric_Pad1.20x1.40mm_HandSolder" (id 2) (at 247.65 73.152 90)
-      (effects (font (size 1.27 1.27)) hide)
-    )
-    (property "Datasheet" "~" (id 3) (at 247.65 74.93 0)
+  (symbol (lib_id "Device:R") (at 251.46 54.61 270) (unit 1)
+    (in_bom yes) (on_board yes)
+    (property "Reference" "R18" (id 0) (at 251.46 57.15 90))
+    (property "Value" "500" (id 1) (at 251.46 59.69 90))
+    (property "Footprint" "Resistor_SMD:R_0805_2012Metric_Pad1.20x1.40mm_HandSolder" (id 2) (at 251.46 52.832 90)
+      (effects (font (size 1.27 1.27)) hide)
+    )
+    (property "Datasheet" "~" (id 3) (at 251.46 54.61 0)
       (effects (font (size 1.27 1.27)) hide)
     )
@@
       (reference "#PWR0136") (unit 1) (value "+3V3") (footprint "")
     )
-    (path "/ad4e483b-3bf5-4c1b-bee3-8f3d5ba2ecf3"
-      (reference "#PWR0137") (unit 1) (value "+3V3") (footprint "")
+    (path "/6764c460-5719-4ae2-9416-3da8b1f102e4"
+      (reference "#PWR0137") (unit 1) (value "Earth") (footprint "")
     )
     (path "/3eadd3f7-174c-4ff3-9be3-e1f91e060ec2"
@@
       (reference "JP1") (unit 1) (value "Jumper_3_Bridged12") (footprint "Jumper:SolderJumper-3_P1.3mm_Bridged12_RoundedPad1.0x1.5mm_NumberLabels")
     )
+    (path "/5b8ae79a-ff7e-45e1-ae08-b9d53dfb1324"
+      (reference "JP2") (unit 1) (value "SolderJumper_2_Open") (footprint "Jumper:SolderJumper-2_P1.3mm_Open_RoundedPad1.0x1.5mm")
+    )
     (path "/5206bb1c-8aa7-4043-9932-e730bc472f2a"

Commit message: added external i2c pins
Parts:
- added J3: Conn_01x04_Male, Connector_PinHeader_2.54mm:PinHeader_1x04_P2.54mm_Vertical, symbol Connector:Conn_01x04_Male
Connections:
- net +3V3: now also J3.2 (Pin_2)
- net Earth: now also J3.1 (Pin_1)
- net SCL: now reaches R6.2, U1.23 (IO15), U3.3 (SCL)
- net SCL: now also J3.3 (Pin_3)
- net SDA: now reaches R7.2, U1.26 (IO4), U3.4 (SDA)
- net SDA: now also J3.4 (Pin_4)
Changed lines of the file:
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@@
+    (stroke (width 0) (type default) (color 0 0 0 0))
+  )
+  (wire (pts (xy 144.78 26.67) (xy 144.78 25.4))
     (stroke (width 0) (type default) (color 0 0 0 0))
   )
@@
     (stroke (width 0) (type default) (color 0 0 0 0))
   )
+  (wire (pts (xy 140.97 30.48) (xy 148.59 30.48))
+    (stroke (width 0) (type default) (color 0 0 0 0))
+  )
   (wire (pts (xy 129.54 78.74) (xy 129.54 81.28))
     (stroke (width 0) (type default) (color 0 0 0 0))
@@
     (stroke (width 0) (type default) (color 0 0 0 0))
   )
+  (wire (pts (xy 146.05 33.02) (xy 148.59 33.02))
+    (stroke (width 0) (type default) (color 0 0 0 0))
+  )
+  (wire (pts (xy 146.05 35.56) (xy 148.59 35.56))
+    (stroke (width 0) (type default) (color 0 0 0 0))
+  )
   (wire (pts (xy 250.19 33.02) (xy 250.19 34.29))
     (stroke (width 0) (type default) (color 0 0 0 0))
@@
     (stroke (width 0) (type default) (color 0 0 0 0))
   )
+  (wire (pts (xy 144.78 25.4) (xy 147.32 25.4))
+    (stroke (width 0) (type default) (color 0 0 0 0))
+  )
   (wire (pts (xy 91.44 149.86) (xy 99.06 149.86))
     (stroke (width 0) (type default) (color 0 0 0 0))
@@
     (stroke (width 0) (type default) (color 0 0 0 0))
   )
+  (wire (pts (xy 147.32 25.4) (xy 147.32 27.94))
+    (stroke (width 0) (type default) (color 0 0 0 0))
+  )
   (wire (pts (xy 26.67 57.15) (xy 26.67 62.23))
     (stroke (width 0) (type default) (color 0 0 0 0))
@@
     (stroke (width 0) (type default) (color 0 0 0 0))
   )
+  (wire (pts (xy 147.32 27.94) (xy 148.59 27.94))
+    (stroke (width 0) (type default) (color 0 0 0 0))
+  )
   (wire (pts (xy 147.32 120.65) (xy 147.32 96.52))
     (stroke (width 0) (type default) (color 0 0 0 0))
@@
   (wire (pts (xy 71.12 104.14) (xy 71.12 120.65))
     (stroke (width 0) (type default) (color 0 0 0 0))
+  )
+  (label "SDA" (at 118.11 55.88 180)
+    (effects (font (size 1.27 1.27)) (justify right bottom))
   )
   (label "SW4-17" (at 67.31 73.66 0)
@@
     (effects (font (size 1.27 1.27)) (justify left bottom))
   )
+  (label "SDA" (at 146.05 35.56 180)
+    (effects (font (size 1.27 1.27)) (justify right bottom))
+  )
   (label "SW6-33" (at 259.08 157.48 180)
     (effects (font (size 1.27 1.27)) (justify right bottom))
@@
     (effects (font (size 1.27 1.27)) (justify left bottom))
   )
+  (label "SCL" (at 118.11 60.96 180)
+    (effects (font (size 1.27 1.27)) (justify right bottom))
+  )
   (label "IRLED-2" (at 67.31 50.8 0)
     (effects (font (size 1.27 1.27)) (justify left bottom))
@@
   (label "SW3-16" (at 67.31 71.12 0)
     (effects (font (size 1.27 1.27)) (justify left bottom))
+  )
+  (label "SCL" (at 146.05 33.02 180)
+    (effects (font (size 1.27 1.27)) (justify right bottom))
   )
   (label "IRLED-2" (at 245.11 54.61 180)
@@
     (pin "1")
     (pin "2")
+  )
+  (symbol (lib_id "Connector:Conn_01x04_Male") (at 153.67 30.48 0) (mirror y) (unit 1)
+    (in_bom yes) (on_board yes) (fields_autoplaced)
+    (property "Reference" "J3" (id 0) (at 154.94 30.4799 0)
+      (effects (font (size 1.27 1.27)) (justify right))
+    )
+    (property "Value" "Conn_01x04_Male" (id 1) (at 154.94 33.0199 0)
+      (effects (font (size 1.27 1.27)) (justify right))
+    )
+    (property "Footprint" "Connector_PinHeader_2.54mm:PinHeader_1x04_P2.54mm_Vertical" (id 2) (at 153.67 30.48 0)
+      (effects (font (size 1.27 1.27)) hide)
+    )
+    (property "Datasheet" "~" (id 3) (at 153.67 30.48 0)
+      (effects (font (size 1.27 1.27)) hide)
+    )
+    (pin "1")
+    (pin "2")
+    (pin "3")
+    (pin "4")
   )
   (symbol (lib_id "Device:C_Polarized") (at 91.44 154.94 0) (unit 1)
@@
     (pin "1")
     (pin "2")
+  )
+  (symbol (lib_id "power:+3V3") (at 140.97 30.48 0) (unit 1)
+    (in_bom yes) (on_board yes) (fields_autoplaced)
+    (property "Reference" "#PWR0139" (id 0) (at 140.97 34.29 0)
+      (effects (font (size 1.27 1.27)) hide)
+    )
+    (property "Value" "+3V3" (id 1) (at 140.97 25.4 0))
+    (property "Footprint" "" (id 2) (at 140.97 30.48 0)
+      (effects (font (size 1.27 1.27)) hide)
+    )
+    (property "Datasheet" "" (id 3) (at 140.97 30.48 0)
+      (effects (font (size 1.27 1.27)) hide)
+    )
+    (pin "1")
   )
   (symbol (lib_id "Interface_Optical:TSOP41xx") (at 214.63 64.77 0) (mirror y) (unit 1)
@@
     (pin "1")
     (pin "2")
+  )
+  (symbol (lib_id "power:Earth") (at 144.78 26.67 0) (unit 1)
+    (in_bom yes) (on_board yes) (fields_autoplaced)
+    (property "Reference" "#PWR0138" (id 0) (at 144.78 33.02 0)
+      (effects (font (size 1.27 1.27)) hide)
+    )
+    (property "Value" "Earth" (id 1) (at 144.78 30.48 0)
+      (effects (font (size 1.27 1.27)) hide)
+    )
+    (property "Footprint" "" (id 2) (at 144.78 26.67 0)
+      (effects (font (size 1.27 1.27)) hide)
+    )
+    (property "Datasheet" "~" (id 3) (at 144.78 26.67 0)
+      (effects (font (size 1.27 1.27)) hide)
+    )
+    (pin "1")
   )
   (symbol (lib_id "RF_Module:ESP32-WROOM-32") (at 49.53 76.2 0) (unit 1)
@@
       (reference "#PWR0137") (unit 1) (value "Earth") (footprint "")
     )
+    (path "/ed385319-554f-4ba7-9d60-89842c6bf432"
+      (reference "#PWR0138") (unit 1) (value "Earth") (footprint "")
+    )
+    (path "/8858f49b-ee7b-4726-8df1-7bda22c8db7f"
+      (reference "#PWR0139") (unit 1) (value "+3V3") (footprint "")
+    )
     (path "/3eadd3f7-174c-4ff3-9be3-e1f91e060ec2"
       (reference "AE1") (unit 1) (value "Antenna 915") (footprint "RF_PCB_Antenna:Micrel_916_ant_6")
@@
       (reference "J2") (unit 1) (value "Wire ANT") (footprint "Connector_PinHeader_1.00mm:PinHeader_1x01_P1.00mm_Vertical")
     )
+    (path "/0dd3171d-103c-4d16-a699-41bf4a04cc8d"
+      (reference "J3") (unit 1) (value "Conn_01x04_Male") (footprint "Connector_PinHeader_2.54mm:PinHeader_1x04_P2.54mm_Vertical")
+    )
     (path "/318e1c86-18c7-41e9-9cf9-b63eea81900c"
